File: daglig.brd (EAGLE design)
At the start: 100 x 80 mm, 25 parts, among them IC1 7805T, Q1 STD17NF03LT4, U1 TLC272D, U2 ATTINY402, U3 MMDT2227-7-F

Commit message: Added todos and resistor values.
Parts:
- R1: value 1m -> 1
- R4: value (none) -> 4k7
- R5, R7: value (none) -> 1k
- R6: value (none) -> 1k8
Changed lines of the file:
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@@
 <attribute name="VALUE" x="41.16" y="13.92" size="1.27" layer="27"/>
 </element>
-<element name="R1" library="rcl" library_urn="urn:adsk.eagle:library:334" package="R2512" package3d_urn="urn:adsk.eagle:package:23545/2" value="1m" x="35.4" y="19.5" smashed="yes" rot="R270">
+<element name="R1" library="rcl" library_urn="urn:adsk.eagle:library:334" package="R2512" package3d_urn="urn:adsk.eagle:package:23545/2" value="1" x="35.4" y="19.5" smashed="yes" rot="R270">
 <attribute name="NAME" x="37.305" y="22.04" size="1.27" layer="25" rot="R270"/>
 <attribute name="POPULARITY" value="0" x="-1.43" y="-8.44" size="1.778" layer="27" rot="R270" display="off"/>
@@
 <attribute name="VALUE" x="43.46" y="31.835" size="1.27" layer="27" rot="R270"/>
 </element>
-<element name="R4" library="rcl" library_urn="urn:adsk.eagle:library:334" package="R0805" package3d_urn="urn:adsk.eagle:package:23553/2" value="" x="39.3" y="41.9" smashed="yes">
+<element name="R4" library="rcl" library_urn="urn:adsk.eagle:library:334" package="R0805" package3d_urn="urn:adsk.eagle:package:23553/2" value="4k7" x="39.3" y="41.9" smashed="yes">
 <attribute name="NAME" x="38.665" y="43.17" size="1.27" layer="25"/>
 <attribute name="POPULARITY" value="86" x="87.56" y="-7.63" size="1.778" layer="27" display="off"/>
@@
 <attribute name="VALUE" x="38.665" y="39.36" size="1.27" layer="27"/>
 </element>
-<element name="R5" library="rcl" library_urn="urn:adsk.eagle:library:334" package="R0805" package3d_urn="urn:adsk.eagle:package:23553/2" value="" x="43.5" y="41.9" smashed="yes">
+<element name="R5" library="rcl" library_urn="urn:adsk.eagle:library:334" package="R0805" package3d_urn="urn:adsk.eagle:package:23553/2" value="1k" x="43.5" y="41.9" smashed="yes">
 <attribute name="NAME" x="42.865" y="43.17" size="1.27" layer="25"/>
 <attribute name="POPULARITY" value="86" x="96.84" y="-7.63" size="1.778" layer="27" display="off"/>
@@
 <attribute name="VALUE" x="42.865" y="39.36" size="1.27" layer="27"/>
 </element>
-<element name="R6" library="rcl" library_urn="urn:adsk.eagle:library:334" package="R0805" package3d_urn="urn:adsk.eagle:package:23553/2" value="" x="33.3" y="40.2" smashed="yes" rot="R180">
+<element name="R6" library="rcl" library_urn="urn:adsk.eagle:library:334" package="R0805" package3d_urn="urn:adsk.eagle:package:23553/2" value="1k8" x="33.3" y="40.2" smashed="yes" rot="R180">
 <attribute name="NAME" x="33.935" y="38.93" size="1.27" layer="25" rot="R180"/>
 <attribute name="POPULARITY" value="86" x="18.06" y="97.35" size="1.778" layer="27" rot="R180" display="off"/>
@@
 <attribute name="VALUE" x="33.935" y="42.74" size="1.27" layer="27" rot="R180"/>
 </element>
-<element name="R7" library="rcl" library_urn="urn:adsk.eagle:library:334" package="R0805" package3d_urn="urn:adsk.eagle:package:23553/2" value="" x="39.3" y="44.1" smashed="yes">
+<element name="R7" library="rcl" library_urn="urn:adsk.eagle:library:334" package="R0805" package3d_urn="urn:adsk.eagle:package:23553/2" value="1k" x="39.3" y="44.1" smashed="yes">
 <attribute name="NAME" x="38.665" y="45.37" size="1.27" layer="25"/>
 <attribute name="POPULARITY" value="86" x="59.62" y="-13.05" size="1.778" layer="27" display="off"/>
